Commit message: init

File: low-level/resources/robots/b1z1/urdf/b1z1.urdf (robot description, URDF)
Before this commit: robot b1z1_description, 29 links, 28 joints
Links:
- link trunk: geometry collision box size=0.647 0.3 0.15; visual mesh filename=/home/lamb/visual_wholebody/low-level/resources/robots/b2w_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 scale=1 1 1

Commit message: init

File: low-level/resources/robots/b1z1/urdf/b1z1.urdf (robot description, URDF)
Before this commit: robot b1z1_description, 29 links, 28 joints
Links:
- link trunk: geometry collision box size=0.647 0.3 0.15; visual mesh filename=/home/lamb/visual_wholebody/low-level/resources/robots/b1z1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 scale=1 1 1

File: low-level/resources/robots/b2z1/urdf/b2z1.urdf (robot description, URDF)
Before this commit: robot b2z1, 34 links, 33 joints
Links:
- link base_link: geometry collision box size=0.5 0.28 0.15; visual mesh filename=/home/lamb/visual_wholebody/low-level/resources/robots/b2z1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
